File: pcb/ExiaNona.sch (EAGLE design)
At the start: 100 parts, among them IC1 ESP32-S3-WROOM-1-N8, IC2 MAX8647ETE+, IC3 LSM6DS3USTR, IC4 NCV8163ASN330T1G, IC6 DG2034EDN-T1-GE4, IC7 BCR421UFD-7, Q1 LTR-4206E, Q2 SI3493DDV-T1-GE3, Q3 IRFML8244TRPBF, Q4 LTR-4206E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

Commit message: change pcb board
Parts:
- removed C17, C18, C8: 0.1u, Capacitor:C1005
- removed U$26, U$29, U$32, U$57: PAD, pad:PAD
- removed Y1: XRCGB40M000F5A00R0, XRCGB40M000F5A00R0:XRCGB40M000F5A00R0
- added C10: 0.1u, Capacitor:C1005
- added IC10: TMUX1108RSVR, TMUX1108RSVR:TMUX1108RSVR
- added IC5: MP6551GQB-P, MP6551GQB-P:MP6551GQB-P
- added IC8: ADS7038IRTER, ADS7038IRTER:ADS7038IRTER
- added Q10, Q11: LTR-4206E, LTR-4206E:LTR-4206E
- added R11, R14: 18, Resistor:R1608
- added R20: 1k, Resistor:R1005
- IC6: value DG2034EDN-T1-GE4 -> MP6551GQB-P; device DG2034EDN-T1-GE4:DG2034EDN-T1-GE4 -> MP6551GQB-P:MP6551GQB-P
- R4: value 10k -> 1k
- U$18, U$22: value TB6614 -> SFH4550; device SSOP16:TB6614 -> LED:SFH4550
Connections:
- removed net ENC_L_A: IC1.GPIO8, U$15.P$4, U$28.P$4
- removed net ENC_L_B: IC1.GPIO9, U$15.P$3, U$28.P$3
- removed net ENC_L_CLK: IC1.GPIO7, U$15.P$5, U$28.P$5
- removed net N$23: U$11.P$1, U$27.P$1, U$3.P$2
- removed net N$33: IC1.XTAL_N, Y1.CRYSTAL_2
- removed net N$36: U$1.P$1, U$18.O2_1, U$18.O2_2, U$32.P$1
- removed net N$37: U$22.O1_1, U$22.O1_2, U$29.P$1, U$8.P$1
- new net ADC_CS: IC1.GPIO17, IC8.!CS
- new net L45_2_CATHODE: IC10.S8, U$18.K
- new net LED_A2: IC1.GPIO10, IC10.A2
- new net N$27: IC5.OUT1_1, IC5.OUT1_2, U$27.P$1
- new net N$28: IC6.OUT1_1, IC6.OUT1_2, U$17.P$1
- new net N$34: C10.1, IC8.DECAP
- new net R45_2_CATHODE: IC10.S7, U$22.K
- new net SEN_L45: IC8.AIN3/GPIO3, Q10.E, R4.2
- new net SEN_R45_2: IC8.AIN2/GPIO2, Q11.E, R20.2
- new net SPI_L_CLK: IC1.GPIO19, IC8.SCLK, U$15.P$5
- new net SPI_L_IN: IC1.GPIO21, IC8.SDO, U$15.P$3
- new net SPI_L_OUT: IC1.GPIO20, IC8.SDI, U$15.P$4
- net +3V3: now also C13.1, IC10.EN, IC10.VDD, IC8.AVDD, IC8.DVDD, Q10.C, Q11.C, R11.1, R14.1; no longer C13.2, C17.2, C18.2, C8.1, IC6.EN, IC6.V+, U$18.STBY, U$18.VCC, U$22.STBY, U$22.VCC
- net A_CW_CCW: now also IC5.IN1; no longer U$18.IN1
- net A_CW_CCW2: now also IC5.IN2; no longer U$18.IN2
- net A_PWM: now also IC5.EN1, IC5.EN2; no longer U$18.PWM
- net BATTERY: now also IC8.AIN7/GPIO7; no longer IC1.GPIO20
- net B_CW_CCW: now also IC6.IN2; no longer U$22.IN1
- net B_CW_CCW1: now also IC6.IN1; no longer U$22.IN2
- net B_PWM: now also IC6.EN1, IC6.EN2; no longer U$22.PWM
- net ENC_L_CS: now also IC1.GPIO18; no longer IC1.GPIO37
- net EN_CLK: now also U$28.P$5
- net EN_MISO: now also U$28.P$3
- net EN_MOSI: now also U$28.P$4
- net GND: now also C10.2, C13.2, IC10.GND, IC10.VSS, IC5.GND, IC8.EP, IC8.GND, R20.1, R4.1; no longer C13.1, C17.1, C18.1, C8.2, IC6.EP, U$18.GND, U$18.PGND1, U$18.PGND2, U$22.GND, U$22.PGND1, U$22.PGND2
- net L45_CATHODE: now also IC10.S6; no longer IC6.S4
- net L90_CATHODE: now also IC10.S5; no longer IC6.S2
- net LED_A0: now also IC1.GPIO8, IC10.A0; no longer IC1.GPIO11, IC6.A0
- net LED_A1: now also IC1.GPIO9, IC10.A1; no longer IC1.GPIO12, IC6.A1
- net LED_EN: now also IC1.GPIO7; no longer IC1.GPIO10
- net LED_SCL: now also IC1.XTAL_32K_P; no longer IC1.GPIO14
- net N$12: now also R14.2, U$22.A; no longer IC1.GPIO19, R4.2
- net N$13: now also U$1.P$1, U$7.P$2; no longer U$17.P$1, U$22.O2_1, U$22.O2_2, U$7.P$1
- net N$2: now also IC6.OUT2_1, IC6.OUT2_2, U$7.P$1, U$8.P$1; no longer IC6.COM, IC7.EP, IC7.OUT
- net N$22: now also U$11.P$1, U$3.P$2; no longer IC1.GPIO21, R4.1
- net N$24: now also IC5.OUT2_1, IC5.OUT2_2, U$3.P$1, U$9.P$1; no longer U$26.P$1, U$57.P$1, U$7.P$2
- net N$32: now also IC10.D, IC7.EP, IC7.OUT; no longer IC1.XTAL_P, Y1.CRYSTAL_1
- net N$6: now also R11.2, U$18.A; no longer U$18.O1_1, U$18.O1_2, U$3.P$1, U$9.P$1
- net R45_CATHODE: now also IC10.S4; no longer IC6.S3
- net R90_CATHODE: now also IC10.S3; no longer IC6.S1
- net SEN_L45_2: now also IC8.AIN1/GPIO1; no longer IC1.GPIO18
- net SEN_L90: now also IC8.AIN6/GPIO6; no longer IC1.XTAL_32K_P
- net SEN_R45: now also IC8.AIN4/GPIO4; no longer IC1.GPIO17
- net SEN_R90: now also IC8.AIN5/GPIO5; no longer IC1.GPIO13
- net VCC: now also IC5.VIN, IC6.VIN; no longer U$18.VM_1, U$18.VM_2, U$22.VM_1, U$22.VM_2
Other:
- moved on the sheet: C12, C13, C4, IC7
